File: hardware/_autosave-flow_monitor.kicad_sch (KiCad schematic)
At the start: 84 parts, among them J1 Conn_01x04_Pin, J2 USB_C_Receptacle_USB2.0_16P, J3 Conn_01x02_Socket, J4 Conn_01x02_Socket, J5 Conn_01x02_Socket, J6 Conn_01x02_Socket, Q1 2N7002, Q2 IRLML6402, Q3 BC807, Q4 BC817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

Commit message: remove comparator circuit from drop detector
Parts:
- removed C10, C12, C7, C9: 100nF, Capacitor_SMD:C_0603_1608Metric, symbol Device:C
- removed C8: 4700nF, Capacitor_SMD:C_0805_2012Metric, symbol Device:C
- removed R12, R13: 47kΩ, Resistor_SMD:R_0603_1608Metric, symbol Device:R
- removed R16, R22, R31: 1MΩ, Resistor_SMD:R_0603_1608Metric, symbol Device:R
- removed R25: 330kΩ, Resistor_SMD:R_0603_1608Metric, symbol Device:R
- removed R26: 10kΩ, Resistor_SMD:R_0603_1608Metric, symbol Device:R
- removed U5: LMV331, Package_TO_SOT_SMD:SOT-23-5, symbol Comparator:LMV331
- added D3: D_TVS, symbol Device:D_TVS
- C16: value 100nF -> 100pF
Connections:
- net GND: now also D3.2 (A2)
- net PD_K: no longer J5.1 (Pin_1), R17.2
- net DROP_INT: no longer names the net of U6.22 (PB10)
- net PD_AC: no longer names the net of R24.2
- net PD_AC: now also J5.1 (Pin_1), R17.2, D3.1 (A1)
Other:
- moved on the sheet: C16, J5, R24
