File: hardware/flow_monitor.kicad_pcb (KiCad board)
At the start: 2 copper layers, 60.3 x 44.9 mm, 80 parts, among them J1 Conn_01x04_Pin, J2 USB_C_Receptacle_USB2.0_16P, J3 Conn_01x02_Socket, J4 Conn_01x02_Socket, J5 Conn_01x02_Socket, Q1 2N7002, Q2 IRLML6402, Q3 BC807, Q4 BC817, Q6 2N7002, SW1 1TS005F-2500-5001, SW2 1TS005F-2500-5001, SW3 1TS005F-2500-5001, SW4 1TS005F-2500-5001, SW5 SW_SPDT, U1 USBLC6-2SC6, U2 BQ25185DLHR, U3 CH340C, U4 TPS631000, U5 LMV331, U6 STM32G030C8Tx, U7 EA_DOGS164W-A, Y1 Crystal

Commit message: hardware: snapshot before power architecture change
Commit current schematic, PCB, and firmware state as a clean
restore point prior to reworking the power supply architecture.
Also adds KiCad autosave/backup patterns to .gitignore.

Co-Authored-By: Claude Sonnet 4.6 <noreply@anthropic.com>
Parts:
- added C7: 100pF, Capacitor_SMD:C_0603_1608Metric, F.Cu at (179.9, 86.1)
- added C8: 100nF, Capacitor_SMD:C_0603_1608Metric, F.Cu at (207.2, 90.2)
- added C9: 0.1uF, Capacitor_SMD:C_0603_1608Metric, F.Cu at (207.2, 92.7)
- added J6: Conn_01x02_Socket, Connector_Wire:SolderWire-0.1sqmm_1x02_P3.6mm_D0.4mm_OD1mm_Relief, F.Cu at (224.4, 80.8)
- added J7: Conn_01x02_Socket_BOT, Connector_Wire:SolderWire-0.1sqmm_1x02_P3.6mm_D0.4mm_OD1mm_Relief, F.Cu at (190.9, 96.6)
- added J8: Conn_01x06_Socket, Connector_FFC-FPC:Jushuo_AFC07-S06FCA-00_1x6-1MP_P0.50_Horizontal, F.Cu at (164.6, 100.2)
- added Q5: 2N7002, Package_TO_SOT_SMD:SOT-23, F.Cu at (169.4, 90.7)
- added R12: 3.3kΩ, Resistor_SMD:R_0603_1608Metric, F.Cu at (179.9, 88.6)
- added R13: 100Ω, Resistor_SMD:R_0603_1608Metric, F.Cu at (179.9, 91.1)
- added R15: 100Ω, Resistor_SMD:R_0603_1608Metric, F.Cu at (179.9, 93.7)
- added R16: 10kΩ, Resistor_SMD:R_0603_1608Metric, F.Cu at (207.2, 95.2)
- added R30: 1800Ω, Resistor_SMD:R_0603_1608Metric, F.Cu at (179.9, 96.2)
- added R32: 100kΩ, Resistor_SMD:R_0603_1608Metric, F.Cu at (179.9, 98.7)
- added R33: 100Ω, Resistor_SMD:R_0603_1608Metric, F.Cu at (179.9, 101.2)
- C16: value 100nF -> 100pF
- C17, C19: value 0.1mF -> 0.1uF
- C18: value 1mF -> 1uF
- J1: value Conn_01x04_Pin -> Conn_01x07_Pin; footprint Connector_PinHeader_2.54mm:PinHeader_1x04_P2.54mm_Vertical -> Connector_PinHeader_2.54mm:PinHeader_1x07_P2.54mm_Vertical
- J5: value Conn_01x02_Socket -> Conn_01x02_Socket_TOP
- SW5: footprint IV_Flow_Monitor_Footprints:UNFINIDHED_SW_Slide_SPDT_SSK12D07VG5 -> IV_Flow_Monitor_Footprints:X_SW_Slide_SPDT_SSK12D07VG5
- moved J1 31.8 mm to (101.5, 86.1), turned to 0 degrees
- moved J3 28.0 mm to (183.3, 81.5)
Connections:
- net /BAT+ renamed BAT+
- net /LED_GATE renamed /LED_GATE_BOT
- C16 pad 2: ADC_IR_DETECTOR -> ADC_IR_DETECTOR_TOP
- J1 pad 4: GND -> UART1_TX
- J2 pad SH: GND -> (no net)
- J4 pad 2: GND -> BAT-
- J5 pad 1: /PD_K -> Net-(J5-Pin_1)
- Q1 pad 2: /IR_LED- -> IR_LED_BOT-
- R17 pad 2: /PD_K -> Net-(J5-Pin_1)
- R24 pad 1: ADC_IR_DETECTOR -> ADC_IR_DETECTOR_TOP
- R24 pad 2: /PD_AC -> Net-(J5-Pin_1)
- R5 pad 2: /IR_LED+ -> IR_LED_BOT+
- R8 pad 2: LED_CTRL -> LED_CTRL_BOT
- U6 pad 14: unconnected-(U6-PA3-Pad14) -> ADC_IR_DETECTOR_TOP
- U6 pad 15: ADC_IR_DETECTOR -> ADC_IR_DETECTOR_BOT
- U6 pad 17: unconnected-(U6-PA6-Pad17) -> LCD_MISO
- U6 pad 22: DROP_INT -> unconnected-(U6-PB10-Pad22)
- U6 pad 42: LED_CTRL -> LED_CTRL_TOP
- U6 pad 43: unconnected-(U6-PB4-Pad43) -> LED_CTRL_BOT
- U6 pad 47: BTN_PLUS -> unconnected-(U6-PB8-Pad47)
- U6 pad 48: BTN_MINUS -> unconnected-(U6-PB9-Pad48)
- U7 pad 15: unconnected-(U7-SOD-Pad15) -> LCD_MISO
Routing:
- net (no net): track 0.00 -> 44.5 mm, vias 0 -> 6
- net LCD_RST: track 33.3 -> 0.00 mm
- net LCD_CS: track 23.5 -> 0.00 mm
- net LED_CTRL: track 23.1 -> 0.00 mm, vias 4 -> 0
- net ADC_IR_DETECTOR: track 21.4 -> 0.00 mm, vias 2 -> 0
- net LCD_MOSI: track 15.9 -> 0.00 mm
- net LCD_SCK: track 15.3 -> 0.00 mm
- net DROP_INT: track 34.8 -> 27.6 mm, vias 5 -> 4
- net IR_LED_BOT-: track 0.00 -> 2.58 mm
- net /IR_LED-: track 2.58 -> 0.00 mm
- net IR_LED_BOT+: track 0.00 -> 2.33 mm
- net /IR_LED+: track 2.33 -> 0.00 mm
- removed copper zone on B.Cu, net GND
